File: PHY_IP101.kicad_sch (KiCad schematic)
At the start: 5 parts, among them U4 ESP32-WROOM-32D

Commit message: Organizando os nomes dos arquivos
Parts:
- C11, C12: value 100nF -> (none); footprint Capacitor_SMD:C_0402_1005Metric_Pad0.74x0.62mm_HandSolder -> (none)
- R13: value 10k -> (none)
- U3: value (none) -> ~
- U4: value ESP32-WROOM-32D -> (none); footprint RF_Module:ESP32-WROOM-32 -> (none)
Changed lines of the file:
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@@
     (in_bom yes) (on_board yes)
     (property "Reference" "C12" (id 0) (at 202.1405 68.4374 0))
-    (property "Value" "100nF" (id 1) (at 203.5706 70.6067 0))
-    (property "Footprint" "Capacitor_SMD:C_0402_1005Metric_Pad0.74x0.62mm_HandSolder" (id 2) (at 197.1548 66.04 0)
+    (property "Value" "" (id 1) (at 203.5706 70.6067 0))
+    (property "Footprint" "" (id 2) (at 197.1548 66.04 0)
       (effects (font (size 1.27 1.27)) hide)
     )
@@
   (symbol (lib_id "power:GNDREF") (at 237.49 58.42 0) (unit 1)
     (in_bom yes) (on_board yes) (fields_autoplaced)
-    (property "Reference" "#PWR033" (id 0) (at 237.49 64.77 0)
+    (property "Reference" "#PWR?" (id 0) (at 237.49 64.77 0)
       (effects (font (size 1.27 1.27)) hide)
     )
-    (property "Value" "GNDREF" (id 1) (at 237.49 63.5 0)
+    (property "Value" "" (id 1) (at 237.49 63.5 0)
       (effects (font (size 1.27 1.27)) hide)
     )
@@
   (symbol (lib_id "power:+3.3V") (at 198.12 54.61 0) (unit 1)
     (in_bom yes) (on_board yes)
-    (property "Reference" "#PWR032" (id 0) (at 198.12 58.42 0)
+    (property "Reference" "#PWR?" (id 0) (at 198.12 58.42 0)
       (effects (font (size 1.27 1.27)) hide)
     )
-    (property "Value" "+3.3V" (id 1) (at 198.12 50.8 0))
+    (property "Value" "" (id 1) (at 198.12 50.8 0))
     (property "Footprint" "" (id 2) (at 198.12 54.61 0)
       (effects (font (size 1.27 1.27)) hide)
@@
       (effects (font (size 1.27 1.27)) (justify left))
     )
-    (property "Value" "10k" (id 1) (at 199.39 60.96 0)
+    (property "Value" "" (id 1) (at 199.39 60.96 0)
       (effects (font (size 1.27 1.27)) (justify left))
     )
@@
   (symbol (lib_id "power:GNDREF") (at 198.12 74.93 0) (unit 1)
     (in_bom yes) (on_board yes) (fields_autoplaced)
-    (property "Reference" "#PWR034" (id 0) (at 198.12 81.28 0)
+    (property "Reference" "#PWR?" (id 0) (at 198.12 81.28 0)
       (effects (font (size 1.27 1.27)) hide)
     )
-    (property "Value" "GNDREF" (id 1) (at 198.12 80.01 0)
+    (property "Value" "" (id 1) (at 198.12 80.01 0)
       (effects (font (size 1.27 1.27)) hide)
     )
@@
     (in_bom yes) (on_board yes)
     (property "Reference" "C11" (id 0) (at 241.5105 51.9274 0))
-    (property "Value" "100nF" (id 1) (at 242.9406 54.0967 0))
-    (property "Footprint" "Capacitor_SMD:C_0402_1005Metric_Pad0.74x0.62mm_HandSolder" (id 2) (at 236.5248 49.53 0)
+    (property "Value" "" (id 1) (at 242.9406 54.0967 0))
+    (property "Footprint" "" (id 2) (at 236.5248 49.53 0)
       (effects (font (size 1.27 1.27)) hide)
     )
@@
   (symbol (lib_id "power:GNDREF") (at 232.41 133.35 0) (unit 1)
     (in_bom yes) (on_board yes) (fields_autoplaced)
-    (property "Reference" "#PWR035" (id 0) (at 232.41 139.7 0)
+    (property "Reference" "#PWR?" (id 0) (at 232.41 139.7 0)
       (effects (font (size 1.27 1.27)) hide)
     )
-    (property "Value" "GNDREF" (id 1) (at 232.41 138.43 0)
+    (property "Value" "" (id 1) (at 232.41 138.43 0)
       (effects (font (size 1.27 1.27)) hide)
     )
@@
       (effects (font (size 1.27 1.27)) (justify left))
     )
-    (property "Value" "" (id 1) (at 112.5094 77.47 0)
+    (property "Value" "~" (id 1) (at 112.5094 77.47 0)
       (effects (font (size 1.27 1.27)) (justify left))
     )
@@
   (symbol (lib_id "power:+3.3V") (at 232.41 45.72 0) (unit 1)
     (in_bom yes) (on_board yes)
-    (property "Reference" "#PWR031" (id 0) (at 232.41 49.53 0)
+    (property "Reference" "#PWR?" (id 0) (at 232.41 49.53 0)
       (effects (font (size 1.27 1.27)) hide)
     )
-    (property "Value" "+3.3V" (id 1) (at 232.41 41.91 0))
+    (property "Value" "" (id 1) (at 232.41 41.91 0))
     (property "Footprint" "" (id 2) (at 232.41 45.72 0)
       (effects (font (size 1.27 1.27)) hide)
@@
       (effects (font (size 1.27 1.27)) (justify left))
     )
-    (property "Value" "ESP32-WROOM-32D" (id 1) (at 233.68 130.81 0)
+    (property "Value" "" (id 1) (at 233.68 130.81 0)
       (effects (font (size 1.27 1.27)) (justify left))
     )
-    (property "Footprint" "RF_Module:ESP32-WROOM-32" (id 2) (at 232.41 133.35 0)
+    (property "Footprint" "" (id 2) (at 232.41 133.35 0)
       (effects (font (size 1.27 1.27)) hide)
     )
