File: POWER_SUPPLY.kicad_sch (KiCad schematic)
At the start: 30 parts, among them CON1 Barrel_Jack_MountingPin, CON2 USB_B_Micro, Q1 AO3401A, U1 AP6503, U2 CP2102N

Commit message: Organizando os nomes dos arquivos
Parts:
- renumbered C7 to C5, C8 to C6, C5 to C7, C6 to C8, R11 to R10, R10 to R11, R5 to R4, R4 to R5

Commit message: Organizando os nomes dos arquivos
Parts:
- C1: value 10nF -> (none); footprint Capacitor_SMD:C_0402_1005Metric_Pad0.74x0.62mm_HandSolder -> (none)
- C10, C6, C8: value 100nF -> (none); footprint Capacitor_SMD:C_0402_1005Metric_Pad0.74x0.62mm_HandSolder -> (none)
- C2: value 22uF/25V -> (none); footprint Capacitor_SMD:C_1206_3216Metric_Pad1.33x1.80mm_HandSolder -> (none)
- C3, C4: value 22uF/16V -> (none); footprint Capacitor_SMD:C_1206_3216Metric_Pad1.33x1.80mm_HandSolder -> (none)
- C5: value 4.7uF -> (none); footprint Capacitor_SMD:C_1206_3216Metric_Pad1.33x1.80mm_HandSolder -> (none)
- C7: value 6,8nF -> (none); footprint Capacitor_SMD:C_0402_1005Metric_Pad0.74x0.62mm_HandSolder -> (none)
- C9: value 10uF -> (none); footprint Capacitor_SMD:C_1206_3216Metric_Pad1.33x1.80mm_HandSolder -> (none)
- CON1: value Barrel_Jack_MountingPin -> (none); footprint Connector_BarrelJack:BarrelJack_GCT_DCJ200-10-A_Horizontal -> (none)
- CON2: value USB_B_Micro -> (none); footprint Connector_USB:USB_Micro-B_GCT_USB3076-30-A -> (none)
- D1, D2: value BAT60A -> (none); footprint Diode_SMD:D_SOD-323 -> (none)
- L1: value 10uH -> (none); footprint Inductor_SMD:L_Bourns-SRN8040_8x8.15mm -> (none)
- Q1: value AO3401A -> (none); footprint Package_TO_SOT_SMD:SOT-23 -> (none)
- R1, R11: value 100k -> (none); footprint Resistor_SMD:R_0402_1005Metric_Pad0.72x0.64mm_HandSolder -> (none)
- R10, R3: value 10k -> (none)
- R12: value 100k -> (none)
- R2: value 26k1 -> (none)
- R4: value 1k -> (none)
- R5: value 6k8 -> (none)
- R6, R7: value 0R -> (none); footprint Resistor_SMD:R_0402_1005Metric_Pad0.72x0.64mm_HandSolder -> (none)
- R8: value 22k -> (none)
- R9: value 47k -> (none)
- U1: value AP6503 -> (none)
- U2: value CP2102N -> (none); footprint Package_DFN_QFN:QFN-28-1EP_5x5mm_P0.5mm_EP3.35x3.35mm -> (none)
